File: Schematics/AD2_extension/Experimental_Kit.kicad_sch (KiCad schematic)
At the start: 11 parts, among them J1 Conn_01x05, J2 AD2, J3 Conn_01x02, J4 Conn_01x02, J5 Conn_01x03, J6 CN7, J7 CN10, J8 AD2, J9 Conn_01x02

Commit message: AD2_extension: on-board level shifters, re-synced PCB, autorouted board
Schematic
- Replace the plug-in BSS138 module (J2/J4) with on-board circuits:
  4x 2N7002 MOSFET shifters (SDA/SCL to LCD, DIO3/DIO5 to PWM) with
  host-side pull-ups on IOREF, TXU0304 fixed-direction SPI shifter
  (VCCA=IOREF, VCCB=3V3), and an IOREF-3V3 header for Feather
- Keypad VCC moved from +3V3 to IOREF (ratiometric ADC readings)
- Add project symbol library (TXU0304PW) and sym-lib-table

PCB
- Sync footprints by UUID after re-annotation, place new parts on the
  back side between the Feather pin rows, mounting holes as H1-H4
- Net classes: Default 0.3 mm, Power 0.6 mm; bottom edge at 120.0 mm
  with copper-to-edge clearance 0.25 mm
- Autoroute with FreeRouting (optimizer threshold 0.1 %), GND pours on
  both layers; DRC: 0 errors, 0 unconnected, schematic parity clean

Co-Authored-By: Claude Fable 5.1 <noreply@anthropic.com>
(cherry picked from commit 84283bcdd4d08d66143eba964df6da12d674042d)
Parts:
- removed J8: AD2, Connector_PinSocket_2.54mm:PinSocket_2x15_P2.54mm_Vertical, symbol Connector_Generic:Conn_02x15_Odd_Even
- added C1, C2: 100nF, Capacitor_SMD:C_0805_2012Metric_Pad1.18x1.45mm_HandSolder, symbol Device:C
- added J12: IOREF, Connector_PinHeader_2.54mm:PinHeader_1x02_P2.54mm_Vertical, symbol Connector_Generic:Conn_01x02
- added J14: SPI, Connector_PinHeader_2.54mm:PinHeader_1x06_P2.54mm_Vertical, symbol Connector_Generic:Conn_01x06
- added J2: Keypad, Connector_PinHeader_2.54mm:PinHeader_1x03_P2.54mm_Vertical, symbol Connector_Generic:Conn_01x03
- added J3: LCD, Connector_PinHeader_2.54mm:PinHeader_1x04_P2.54mm_Vertical, symbol Connector_Generic:Conn_01x04
- added J5, J6: PWM, Connector_PinHeader_2.54mm:PinHeader_1x03_P2.54mm_Vertical, symbol Connector_Generic:Conn_01x03
- added Q1, Q2, Q3, Q4: 2N7002, Package_TO_SOT_SMD:SOT-23, symbol Transistor_FET:2N7002
- added R1, R3, R5, R6, R7, R8: 10k, Resistor_SMD:R_0805_2012Metric_Pad1.20x1.40mm_HandSolder, symbol Device:R
- added R2, R4: 4.7k, Resistor_SMD:R_0805_2012Metric_Pad1.20x1.40mm_HandSolder, symbol Device:R
- added U1: TXU0304PW, Package_SO:TSSOP-14_4.4x5mm_P0.65mm, symbol AD2_extension:TXU0304PW
- A1: footprint Module:Arduino_UNO_R3 -> AD2_extension:Arduino_UNO_R3_ShieldHeaders
- J11: renamed from J6; footprint Connector_PinSocket_2.54mm:PinSocket_2x19_P2.54mm_Vertical -> AD2_extension:PinSocket_2x19_P2.54mm_Vertical_Mirrored
- J13: renamed from J7; footprint Connector_PinSocket_2.54mm:PinSocket_2x19_P2.54mm_Vertical -> AD2_extension:PinSocket_2x19_P2.54mm_Vertical_Mirrored
- J7: renamed from J3; value Conn_01x02 -> AREF
- J9: renamed from J4; value Conn_01x02 -> W1
- renumbered J5 to J1, J2 to J10, J1 to J4, J9 to J8
Connections:
- net +3V3: now also C2.2, J12.2 (Pin_2), J14.2 (Pin_2), U1.14 (VCCB), U1.8 (OE)
- net +5V: now also J3.2 (Pin_2), J5.2 (Pin_2), J6.2 (Pin_2), R1.1, R3.1, R5.1, R7.1
- net A0: now also J2.3 (Pin_3)
- net DIO10: now also U1.4 (A3)
- net DIO11: now also U1.3 (A2)
- net DIO12: now also U1.5 (A4Y)
- net DIO13: now also U1.2 (A1)
- net DIO3: now also Q3.2 (S), R6.1
- net DIO5: now also Q4.2 (S), R8.1
- net GND: now also C1.1, C2.1, J14.1 (Pin_1), J2.1 (Pin_1), J3.1 (Pin_1), J5.1 (Pin_1), J6.1 (Pin_1), U1.7 (GND)
- net IOREF: now also C1.2, J12.1 (Pin_1), J2.2 (Pin_2), Q1.1 (G), Q2.1 (G), Q3.1 (G), Q4.1 (G), R2.2, R4.2, R6.2, R8.2, U1.1 (VCCA)
- net SCL/A5: now also Q2.2 (S), R4.1
- net SDA/A4: now also Q1.2 (S), R2.1
- new net DIO3_5V: J5.3 (Pin_3), Q3.3 (D), R5.2
- new net DIO5_5V: J6.3 (Pin_3), Q4.3 (D), R7.2
- new net LCD_SCL: J3.4 (Pin_4), Q2.3 (D), R3.2
- new net LCD_SDA: J3.3 (Pin_3), Q1.3 (D), R1.2
- new net SPI_CS: J14.3 (Pin_3), U1.11 (B3Y)
- new net SPI_MISO: J14.5 (Pin_5), U1.10 (B4)
- new net SPI_MOSI: J14.6 (Pin_6), U1.12 (B2Y)
- new net SPI_SCK: J14.4 (Pin_4), U1.13 (B1Y)
Other:
- note added: "IOREF: UNO=5V, Nucleo=3.3V, Feather: no IOREF pin -> close JP1 (IOREF=3V3)"
- note added: "Level shifter (on-board): host IOREF <-> 5V (I2C LCD, PWM servo) / 3V3 (SPI)"
- note added: "Q1-Q4: bidirectional MOSFET level shifter (NXP AN10441). Gate + host pull-up = IOREF, far side = +5V"
- note added: "U1 TXU0304: A1-A3 -> B1-B3 (SCK, MOSI, CS), B4 -> A4 (MISO). VCCA = IOREF, VCCB = +3V3"
- moved on the sheet: J10, J7, J8, J9
