File: Schematics/AD2_extension/Experimental_Kit.kicad_sch (KiCad schematic)
At the start: 31 parts, among them J1 Conn_01x03, J10 AD2, J11 CN7, J12 IOREF, J13 CN10, J14 SPI, J2 Keypad, J3 LCD, J4 Conn_01x05, J5 PWM, J6 PWM, J7 AREF, J8 Conn_01x02, J9 W1, Q1 2N7002, Q2 2N7002, Q3 2N7002, Q4 2N7002, U1 TXU0304PW

Commit message: Add Quartus_labs
Parts:
- removed J1: Conn_01x03, Connector_PinHeader_2.54mm:PinHeader_1x03_P2.54mm_Vertical, symbol Connector_Generic:Conn_01x03
- removed J4: Conn_01x05, Connector_PinHeader_2.54mm:PinHeader_1x05_P2.54mm_Vertical, symbol Connector_Generic:Conn_01x05
- added J1: Conn_01x04, Connector_PinHeader_2.54mm:PinHeader_1x04_P2.54mm_Vertical, symbol Connector_Generic:Conn_01x04
- added J4: Conn_01x06, symbol Connector_Generic:Conn_01x06
Connections:
- net +3V3: now also J1.2 (Pin_2), J4.2 (Pin_2); no longer C2.2, J14.2 (Pin_2), U1.14 (VCCB)
- net +5V: now also J14.2 (Pin_2), U1.14 (VCCB)
- net DIO10: now also J4.3 (Pin_3)
- net GND: now also J1.1 (Pin_1), J4.1 (Pin_1)
- net SCL: now also J1.3 (Pin_3)
- net SDA: now also J1.4 (Pin_4)
- net at MS1.11 (GPIOSCK): now also J4.6 (Pin_6)
- net at MS1.12 (GPIOMOSI): now also J4.5 (Pin_5)
- net at MS1.13 (GPIOMISO): now also J4.4 (Pin_4)
- no-connect marks 47 -> 53
