File: Schematics/AD2_extension/Experimental_Kit.kicad_pcb (KiCad board)
At the start: 2 copper layers, 69.7 x 76.4 mm, 35 parts, among them J1 Conn_01x03, J10 AD2, J11 CN7, J12 IOREF, J13 CN10, J14 SPI, J2 Keypad, J3 LCD, J4 Conn_01x05, J5 PWM, J6 PWM, J7 AREF, J8 Conn_01x02, J9 W1, Q1 2N7002, Q2 2N7002, Q3 2N7002, Q4 2N7002, U1 TXU0304PW

Commit message: Add Quartus_labs
Parts:
- J1: value Conn_01x03 -> Conn_01x04; footprint Connector_PinHeader_2.54mm:PinHeader_1x03_P2.54mm_Vertical -> Connector_PinHeader_2.54mm:PinHeader_1x04_P2.54mm_Vertical
- J4: value Conn_01x05 -> Conn_01x06
- moved J4 45.6 mm to (94.9, 112.5), turned to 90 degrees
- moved J14 41.9 mm to (120.9, 112.5), turned to 90 degrees
- moved J1 35.7 mm to (81.4, 108.5)
- moved J3 6.59 mm to (81.5, 105.0), turned to 90 degrees
Connections:
- C2 pad 2: +3V3 -> unconnected-(C2-Pad2)
- J1 pad 1: /SDA -> GND
- J1 pad 2: /SCL -> +3V3
- J1 pad 3: GND -> /SCL
- J14 pad 2: +3V3 -> +5V
- J4 pad 1: Net-(J4-Pin_1) -> GND
- J4 pad 2: Net-(J4-Pin_2) -> +3V3
- J4 pad 3: Net-(J4-Pin_3) -> /DIO10
- J4 pad 4: /DIO10 -> Net-(J4-Pin_4)
- J4 pad 5: GND -> Net-(J4-Pin_5)
- MS1 pad 11: Net-(J4-Pin_1) -> Net-(J4-Pin_6)
- MS1 pad 12: Net-(J4-Pin_2) -> Net-(J4-Pin_5)
- MS1 pad 13: Net-(J4-Pin_3) -> Net-(J4-Pin_4)
- U1 pad 14: +3V3 -> +5V
Routing:
- net GND: track 318.0 -> 46.5 mm
- net +5V: track 162.4 -> 8.78 mm, vias 4 -> 0
- net /DIO10: track 139.5 -> 49.7 mm, vias 2 -> 0
- net /LCD_SDA: track 72.1 -> 5.01 mm, vias 1 -> 0
- net /LCD_SCL: track 66.6 -> 0.00 mm, vias 2 -> 0
- net /SPI_MOSI: track 59.1 -> 0.01 mm, vias 1 -> 0
- net +3V3: track 83.3 -> 44.4 mm, vias 4 -> 0
- net /SPI_MISO: track 36.7 -> 0.00 mm, vias 1 -> 0
- net /SPI_CS: track 31.4 -> 0.00 mm, vias 1 -> 0
- net /SPI_SCK: track 30.2 -> 0.00 mm, vias 1 -> 0
- net /DIO11: track 98.1 -> 79.7 mm
- net Net-(J4-Pin_1): track 12.6 -> 0.00 mm
- net Net-(J4-Pin_3): track 12.3 -> 0.00 mm
- net Net-(J4-Pin_2): track 11.9 -> 0.00 mm
- net /DIO9: track 63.7 -> 62.6 mm
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- removed copper zone on F.Cu, net GND
